Commit message: change lifter ankle_joint angle limit 90 -> 65

File: aero_shop/typeC_lifter/urdf/lifter.urdf.xacro (robot description, xacro)
@@ -169,5 +169,5 @@
       <origin xyz="0 0 0.05" rpy="0 0 0"/>
       <axis   xyz="0 -1 0"/>
-      <limit effort="10000" lower="0" upper="1.5707" velocity="0.5" />
+      <limit effort="10000" lower="0" upper="1.13446" velocity="0.5" />
       <dynamics damping="0.2" friction="0" />
     </joint>
@@ -181,5 +181,5 @@
       <axis   xyz="0 -1 0"/>
       <mimic joint="ankle_joint" multiplier="-1" offset="0" />
-      <limit effort="10000" upper="0" lower="-1.5707" velocity="0.5" /> <!-- just invert of ankle_joint -->
+      <limit effort="10000" upper="0" lower="-1.13446" velocity="0.5" /> <!-- just invert of ankle_joint -->
     </joint>
 <!-- redundant -->
